Commit message: SLAM ve Navigasyon entegrasyonu tamamlandi. Harita ve URDF duzeltmeleri eklendi.

File: urdf/robot.urdf.xacro (robot description, xacro)
@@ -1,13 +1,8 @@
 <?xml version="1.0"?>
 <robot xmlns:xacro="http://www.ros.org/wiki/xacro"  name="my_robot">
-    <material name="white">
-        <color rgba="1 1 1 1" />
-    </material>
-    <material name="blue">
-        <color rgba="0.2 0.2 1 1"/>
-    </material>
-    <material name="black">
-        <color rgba="0 0 0 1"/>
-    </material>
+    <material name="white"><color rgba="1 1 1 1" /></material>
+    <material name="blue"><color rgba="0.2 0.2 1 1"/></material>
+    <material name="black"><color rgba="0 0 0 1"/></material>
+    <material name="red"><color rgba="1 0 0 1"/></material>
     <xacro:macro name="inertial_box" params="mass x y z *origin">
         <inertial>
@@ -37,6 +32,11 @@
         </inertial>
     </xacro:macro>
-    <link name="base_link">
-    </link>
+    <link name="base_footprint"/>
+    <joint name="base_joint" type="fixed">
+        <parent link="base_footprint"/>
+        <child link="base_link"/>
+        <origin xyz="0 0 0.10"/>
+    </joint>
+    <link name="base_link"></link>
     <joint name="chassis_joint" type="fixed">
         <parent link="base_link"/>
@@ -47,16 +47,12 @@
         <visual>
             <origin xyz="0.15 0 0.075"/>
-            <geometry>
-                <box size="0.3 0.3 0.15"/>
-            </geometry>
+            <geometry><box size="0.3 0.3 0.15"/></geometry>
             <material name="white"/>
         </visual>
         <collision>
             <origin xyz="0.15 0 0.075"/>
-            <geometry>
-                <box size="0.3 0.3 0.15"/>
-            </geometry>
+            <geometry><box size="0.3 0.3 0.15"/></geometry>
         </collision>
-        <xacro:inertial_box mass="0.5" x="0.3" y="0.3" z="0.15">
+        <xacro:inertial_box mass="1.0" x="0.3" y="0.3" z="0.15">
             <origin xyz="0.15 0 0.075" rpy="0 0 0"/>
         </xacro:inertial_box>
@@ -70,15 +66,11 @@
     <link name="left_wheel">
         <visual>
-            <geometry>
-                <cylinder radius="0.05" length="0.04"/>
-            </geometry>
+            <geometry><cylinder radius="0.05" length="0.04"/></geometry>
             <material name="blue"/>
         </visual>
         <collision>
-            <geometry>
-                <cylinder radius="0.05" length="0.04"/>
-            </geometry>
+            <geometry><cylinder radius="0.05" length="0.04"/></geometry>
         </collision>
-        <xacro:inertial_cylinder mass="0.1" length="0.04" radius="0.05">
+        <xacro:inertial_cylinder mass="0.2" length="0.04" radius="0.05">
             <origin xyz="0 0 0" rpy="0 0 0"/>
         </xacro:inertial_cylinder>
@@ -92,15 +84,11 @@
     <link name="right_wheel">
         <visual>
-            <geometry>
-                <cylinder radius="0.05" length="0.04"/>
-            </geometry>
+            <geometry><cylinder radius="0.05" length="0.04"/></geometry>
             <material name="blue"/>
         </visual>
         <collision>
-            <geometry>
-                <cylinder radius="0.05" length="0.04"/>
-            </geometry>
+            <geometry><cylinder radius="0.05" length="0.04"/></geometry>
         </collision>
-        <xacro:inertial_cylinder mass="0.1" length="0.04" radius="0.05">
+        <xacro:inertial_cylinder mass="0.2" length="0.04" radius="0.05">
             <origin xyz="0 0 0" rpy="0 0 0"/>
         </xacro:inertial_cylinder>
@@ -113,13 +101,9 @@
     <link name="caster_wheel">
         <visual>
-            <geometry>
-                <sphere radius="0.05"/>
-            </geometry>
+            <geometry><sphere radius="0.05"/></geometry>
             <material name="black"/>
         </visual>
         <collision>
-            <geometry>
-                <sphere radius="0.05"/>
-            </geometry>
+            <geometry><sphere radius="0.05"/></geometry>
         </collision>
         <xacro:inertial_sphere mass="0.1" radius="0.05">
@@ -129,16 +113,23 @@
     <gazebo reference="caster_wheel">
         <material>Gazebo/Black</material>
-        <mu1 value="0.001"/>
-        <mu2 value="0.001"/>
+        <mu1>0.00001</mu1>
+        <mu2>0.00001</mu2>
+        <minDepth>0.001</minDepth>
+    </gazebo>
+    <gazebo reference="left_wheel">
+        <material>Gazebo/Blue</material>
+        <mu1>1.0</mu1>
+        <mu2>1.0</mu2>
+        <minDepth>0.001</minDepth>
+    </gazebo>
+    <gazebo reference="right_wheel">
+        <material>Gazebo/Blue</material>
+        <mu1>1.0</mu1>
+        <mu2>1.0</mu2>
+        <minDepth>0.001</minDepth>
     </gazebo>
     <gazebo reference="chassis">
         <material>Gazebo/White</material>
     </gazebo>
-    <gazebo reference="left_wheel">
-        <material>Gazebo/Blue</material>
-    </gazebo>
-    <gazebo reference="right_wheel">
-        <material>Gazebo/Blue</material>
-    </gazebo>
     <xacro:include filename="gazebo_control.xacro" />
     <xacro:include filename="lidar.xacro" />
